File: Final Project/Object Test Board/object01.brd (EAGLE design)
At the start: 100 x 80 mm, 18 parts, among them IC1 7805T, IC2 ATMEGA328P

Commit message: small edits to board
Parts:
- added 13LED, LED4, LED5, LED6: (no value), led:LED5MM
- added JP10, JP11, JP12: (no value), adafruit:1X01
- added LED7: RGBLED_CA-5MM, adafruit:LED5MMRGB
- added PH1: V1060_21, photo-elements:TO-5_V10
- added R1, R10, R220, R3, R4, R6, R7, R8, R9: (no value), resistor:0207/10
- added TM1: (no value), adafruit:TRIM-3386
Connections:
- new net N$10: LED7.1, R6.2
- new net N$11: LED7.3, R9.2
- new net N$12: LED5.K, R3.1
- new net N$13: LED4.K, R1.1
- new net N$14: LED6.K, R4.1
- new net N$16: IC2.14, JP12.1
- new net N$17: IC2.5, LED6.A
- new net N$18: IC2.11, LED5.A
- new net N$19: IC2.12, LED4.A
- new net N$20: IC2.23, TM1.2
- new net N$21: IC2.24, PH1.2, R8.2
- new net N$22: IC2.13, JP11.1
- new net N$23: IC2.4, R7.1
- new net N$24: IC2.6, JP10.1, R7.2
- new net N$25: LED7.4, R10.2
- new net N$26: 13LED.K, R220.2
- new net N$27: IC2.15, R6.1
- new net N$28: IC2.16, R9.1
- net +5V: now also PH1.1, TM1.1
- net GND: now also LED7.2, R1.2, R220.1, R3.2, R4.2, R8.1, TM1.3
- net N$4: now also R10.1
- net N$6: now also 13LED.A
Routing:
- net GND: track 181.9 -> 269.1 mm
- net N$6: track 4.33 -> 71.6 mm
- net +5V: track 89.3 -> 127.1 mm
- net N$21: track 0.00 -> 30.5 mm
- net N$17: track 0.00 -> 22.6 mm
- net N$24: track 0.00 -> 22.3 mm
- net N$13: track 0.00 -> 15.9 mm
- net N$19: track 0.00 -> 12.4 mm
- net N$4: track 4.38 -> 16.0 mm
- net N$20: track 0.00 -> 11.3 mm
- net N$28: track 0.00 -> 10.3 mm
- net N$18: track 0.00 -> 10.0 mm
- net N$16: track 0.00 -> 9.37 mm
- net N$25: track 0.00 -> 9.30 mm
- net N$22: track 0.00 -> 9.02 mm
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